File: Project Architecture.kicad_sch (KiCad schematic)
At the start: 0 parts

Commit message: [sch] first release of the schematic
Other:
- sheet Section A - Title A renamed Sec A - Shift Register Screw Interface
- sheet Section B - Title B renamed Sec B - Shift Register
- added sheet Sec C - LED Display (Sec C - LED Display.kicad_sch)
- sheet Sec A - Shift Register Screw Interface: file Section A - Title A.kicad_sch -> Sec A - SR Screw Interface.kicad_sch
- sheet Sec A - Shift Register Screw Interface ports: added SR_CLK, SR_LATCH, SR_SDI; removed none
- sheet Sec B - Shift Register: file Section B - TItle B.kicad_sch -> Sec B - Shift Register.kicad_sch
- sheet Sec B - Shift Register ports: added L[1..16], RS_CLK, RS_LATCH, RS_SDI; removed none
- note added: "Page 6"
