File: Sec A - SR Screw Interface.kicad_sch (KiCad schematic)
At the start: 1 part, among them U1 B-B Interface

Commit message: preliminary pcb version
Parts:
- U1: footprint (none) -> __Sienkiewicz:Sienkiewicz
Connections:
- net SR_CLK: now also U1.4 (CLK); no longer U1.1 (CLK)
- net SR_SDI: now also U1.1 (SDI); no longer U1.4 (SDI)
Changed lines of the file:
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@@
 	(hierarchical_label "SR_CLK"
 		(shape output)
-		(at 142.24 68.58 180)
+		(at 142.24 73.66 180)
 		(effects
 			(font
@@
 	(hierarchical_label "SR_SDI"
 		(shape output)
-		(at 142.24 73.66 180)
+		(at 142.24 68.58 180)
 		(effects
 			(font
@@
 			)
 		)
-		(property "Footprint" ""
+		(property "Footprint" "__Sienkiewicz:Sienkiewicz"
 			(at 160.02 71.12 0)
 			(effects
