File: Sec B - Shift Register.kicad_sch (KiCad schematic)
At the start: 6 parts, among them U2 STP16CP05M

Commit message: preliminary pcb version
Parts:
- R1: footprint (none) -> Resistor_SMD:R_1206_3216Metric
Changed lines of the file:
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@@
 		(dnp no)
 		(property "Reference" "R1"
-			(at 124.46 99.06 90)
+			(at 127 99.06 90)
 			(effects
 				(font
@@
 		)
 		(property "Value" "1k5"
-			(at 129.54 99.06 90)
+			(at 132.08 99.06 90)
 			(effects
 				(font
@@
 			)
 		)
-		(property "Footprint" ""
+		(property "Footprint" "Resistor_SMD:R_1206_3216Metric"
 			(at 129.54 96.52 0)
 			(effects
