File: Sec C - LED Display.kicad_sch (KiCad schematic)
At the start: 16 parts

Commit message: preliminary pcb version
Parts:
- D1, D10, D11, D12, D13, D14, D15, D16, D2, D3, D4, D5, D6, D7, D8, D9: footprint (none) -> LED_SMD:LED_1206_3216Metric
