File: Sienkiewicz_LED.kicad_pcb (KiCad board)
At the start: 2 copper layers, 38 x 38 mm, 25 parts, among them U1 B-B Interface, U2 STP16CP05M

Commit message: Update Outputs (release)
Other:
- board text added: "0.035mm (1.00oz)"
- board text added: "1.5mm"
- board text added: "Total thickness: 1.61mm"
- board text removed: "0.07mm (2.00oz)"
- board text removed: "1.48mm"
- board text removed: "Total thickness: 1.66mm"

Commit message: silkcreen version bump to 2.1.1
Other:
- board text added: "SW:2.1.1"
- board text removed: "SW:2.1.X"

Commit message: pcb silkscreen version fix
Other:
- board text added: "HW:2.1.1"
- board text added: "SW:2.1.X"
- board text removed: "HW:2.1.0"
- board text removed: "SW:2.1.1"
Changed lines of the file:
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@@
 		)
 	)
-	(gr_text "HW:2.1.0"
+	(gr_text "HW:2.1.1"
 		(at 135.5 96 0)
 		(layer "B.SilkS")
@@
 		)
 	)
-	(gr_text "SW:2.1.1"
+	(gr_text "SW:2.1.X"
 		(at 135.5 98 0)
 		(layer "B.SilkS")
